Commit message: returned to old urdf

File: hera_description/urdf/hera_description.urdf (robot description, URDF)
Before this commit: robot hera_description, 20 links, 19 joints
Links:
- link base_link: mass 20 -> 99.5369630102893
Joints:
- joint head_joint: axis 0 0 0 -> 0 0 1; limit (none) -> lower=-1.2 upper=1.2 effort=3 velocity=3; type fixed -> revolute
- joint joint_1: limit effort=10.6 velocity=5 -> lower=-2.24 upper=2.24 effort=10.6 velocity=5; type fixed -> revolute
- joint joint_2: limit effort=10.6 velocity=5 -> lower=-3.14 upper=3.14 effort=10.6 velocity=5; origin xyz=0.048 0 0.0215 rpy=3.1416 -0.8154 -3.1416 -> xyz=0.048 0 0.0215 rpy=3.1416 -1.1781 -3.1416; type fixed -> revolute
- joint joint_3: limit effort=10.6 velocity=5 -> lower=-2.24 upper=2.24 effort=10.6 velocity=5; type fixed -> revolute
- joint joint_4: limit effort=10.6 velocity=5 -> lower=-5.14 upper=1.14 effort=10.6 velocity=5; origin xyz=0.0215 0.0001535 -0.048 rpy=8.3578E-18 -0.4681 -2.9674E-16 -> xyz=0.0215 0.0001535 -0.048 rpy=8.3578E-18 -0.3927 -2.9674E-16; type fixed -> revolute
- joint joint_5: limit effort=10.6 velocity=5 -> lower=-2.24 upper=2.24 effort=10.6 velocity=5; origin xyz=0.14525 0 0 rpy=-0.0090 1.4438E-31 -8.5251E-17 -> xyz=0.14525 0 0 rpy=-1.4604E-16 1.4438E-31 -8.5251E-17; type fixed -> revolute
- joint joint_6: limit effort=10.6 velocity=5 -> lower=-3.14 upper=3.14 effort=10.6 velocity=5; origin xyz=0.0375 0 0 rpy=0 2.6196 0 -> xyz=0.0375 0 0 rpy=0 2.6042E-31 0; type fixed -> revolute
- joint kinect_joint: limit (none) -> lower=0 upper=1.57 effort=3 velocity=3; type fixed -> revolute
