Commit message: changes urdf

File: hera_description/urdf/actuators/torso.urdf.xacro (robot description, xacro)
@@ -95,11 +95,11 @@
     </joint>
     <!-- should be revolute -->
-    <joint name="joint_${name}_to_${name}_sensor_plat" type="fixed">
+    <joint name="joint_${name}to${name}_sensor_plat" type="revolute">
       <origin xyz="0.09 0 0.46" rpy="0 ${55 *(M_PI/180)} 0"/> <!-- rpy="0 0 0" -->
       <parent link="${name}"/>
       <child link="${name}_sensor_plat"/>
-      <!-- <axis xyz="0 1 0"/> -->
-      <!-- <limit effort="${torso_sensor_plat_effort}" velocity="${torso_sensor_plat_velocity}"
-        lower="0.0" upper="${M_PI/2}"/> -->
+      <axis xyz="0 1 0"/>
+      <limit effort="${torso_sensor_plat_effort}" velocity="${torso_sensor_plat_velocity}"
+        lower="-1.0216" upper="-0.6592" />
     </joint>
     <!-- <transmission name="tran_${name}_sensor_plat">

Commit message: RPY parameter

File: hera_description/urdf/actuators/torso.urdf.xacro (robot description, xacro)
@@ -96,5 +96,5 @@
     <!-- should be revolute -->
     <joint name="joint_${name}to${name}_sensor_plat" type="revolute">
-      <origin xyz="0.09 0 0.46" rpy="0 ${55 *(M_PI/180)} 0"/> <!-- rpy="0 0 0" -->
+      <origin xyz="0.09 0 0.46" rpy="0 0 0"/> <!-- rpy="0 0 0" -->
       <parent link="${name}"/>
       <child link="${name}_sensor_plat"/>

Commit message: Voltando para fixo o kinect

File: hera_description/urdf/actuators/torso.urdf.xacro (robot description, xacro)
@@ -102,11 +102,12 @@
     </joint>
     <!-- should be revolute -->
-    <joint name="joint_${name}_to_${name}_sensor_plat" type="revolute">
+    <!-- should be revolute -->
+    <joint name="joint_${name}_to_${name}_sensor_plat" type="fixed">
       <origin xyz="0.09 0 0.46" rpy="0 0 0"/> <!-- rpy="0 0 0" -->
       <parent link="${name}"/>
       <child link="${name}_sensor_plat"/>
-      <axis xyz="0 1 0"/> -->
-      <limit effort="${torso_sensor_plat_effort}" velocity="${torso_sensor_plat_velocity}"
-        lower="0.0" upper="1.57"/>
+      <!-- <axis xyz="0 1 0"/> -->
+      <!-- <limit effort="${torso_sensor_plat_effort}" velocity="${torso_sensor_plat_velocity}"
+        lower="0.0" upper="${M_PI/2}"/> -->
     </joint>
     <!-- <transmission name="tran_${name}_sensor_plat">

Commit message: Setting PID for manipulator

File: hera_description/urdf/actuators/torso.urdf.xacro (robot description, xacro)
@@ -20,5 +20,5 @@
   <xacro:property name="pole_size_y"       value="0.06"/>
   <xacro:property name="pole_size_z"       value="1.00"/>
-  <xacro:property name="sensor_plat_mass"             value="0.01"/>
+  <xacro:property name="sensor_plat_mass"             value="1.0"/>
   <xacro:property name="sensor_plat_size_x"           value="0.10"/>
   <xacro:property name="sensor_plat_size_y"           value="0.12"/>
