Commit message: Changed robot base mass

File: hera_description/urdf/actuators/base.urdf.xacro (robot description, xacro)
@@ -4,5 +4,5 @@
        xmlns:interface="http://playerstage.sourceforge.net/gazebo/xmlschema/#interface"
        xmlns:xacro="http://ros.org/wiki/xacro">
-  <xacro:property name="base_mass"      value="20.0"/>
+  <xacro:property name="base_mass"      value="99.9"/>
   <xacro:property name="base_size_x"    value="0.50"/>
   <xacro:property name="base_size_y"    value="0.30"/>

Commit message: Higher gripper

File: hera_description/urdf/actuators/base.urdf.xacro (robot description, xacro)
@@ -4,5 +4,5 @@
        xmlns:interface="http://playerstage.sourceforge.net/gazebo/xmlschema/#interface"
        xmlns:xacro="http://ros.org/wiki/xacro">
-  <xacro:property name="base_mass"      value="50.0"/>
+  <xacro:property name="base_mass"      value="20.0"/>
   <xacro:property name="base_size_x"    value="0.50"/>
   <xacro:property name="base_size_y"    value="0.30"/>

File: hera_description/urdf/actuators/gripper/robotiq-3f-gripper_articulated_macro.xacro (robot description, xacro)
@@ -15,5 +15,5 @@
 			<visual>
 				<geometry>
-                    <mesh filename="package://hera_description/meshes/gripper_meshes/visual/palm.dae" scale= "0.6 0.6 0.6" />
+                    <mesh filename="package://hera_description/meshes/gripper_meshes/visual/palm.dae" scale= "0.7 0.7 0.7" />
 				</geometry>
 				<material name="white">
@@ -23,5 +23,5 @@
 			<collision>
 				<geometry>
-                    <mesh filename="package://hera_description/meshes/gripper_meshes/collision/palm.STL" scale= "0.6 0.6 0.6" />
+                    <mesh filename="package://hera_description/meshes/gripper_meshes/collision/palm.STL" scale= "0.7 0.7 0.7" />
 				</geometry>
 				<material name="yellow">
@@ -46,15 +46,15 @@
 			<parent link="${prefix}palm"/>
 			<child link="${prefix}finger_1_link_0"/>
-			<origin xyz="-0.0255 0.005 0.0225" rpy="0 3.1416 -1.57"/>
+			<origin xyz="-0.0255 0.01 0.0225" rpy="0 3.1416 -1.57"/>
 		</joint>
 		<joint name="${prefix}palm_finger_2_joint" type="fixed">
 			<parent link="${prefix}palm"/>
 			<child link="${prefix}finger_2_link_0"/>
-			<origin xyz="-0.0255 0.005 -0.0225" rpy="0 3.1416 -1.57"/>
+			<origin xyz="-0.0255 0.01 -0.0225" rpy="0 3.1416 -1.57"/>
 		</joint>
 		<joint name="${prefix}palm_finger_middle_joint" type="fixed">
 			<parent link="${prefix}palm"/>
 			<child link="${prefix}finger_middle_link_0"/>
-			<origin xyz="0.0255 0.005 0" rpy="0 0 1.57"/>
+			<origin xyz="0.0255 0.01 0" rpy="0 0 1.57"/>
 		</joint>
 		<joint name="${prefix}palm_tool0" type="fixed">

File: hera_description/urdf/actuators/gripper/robotiq-3f-gripper_finger_articulated_macro.xacro (robot description, xacro)
@@ -12,5 +12,5 @@
 				<origin xyz="0.020 0 0" rpy="0 0 0"/>
 				<geometry>
-                    <mesh filename="package://hera_description/meshes/gripper_meshes/visual/link_0.dae" scale= "0.6 0.6 0.6" />
+                    <mesh filename="package://hera_description/meshes/gripper_meshes/visual/link_0.dae" scale= "0.7 0.7 0.7" />
 				</geometry>
 				<material name="white">
@@ -21,5 +21,5 @@
 				<origin xyz="0.020 0 0" rpy="0 0 0"/>
 				<geometry>
-                    <mesh filename="package://hera_description/meshes/gripper_meshes/collision/link_0.STL" scale= "0.6 0.6 0.6" />
+                    <mesh filename="package://hera_description/meshes/gripper_meshes/collision/link_0.STL" scale= "0.7 0.7 0.7" />
 				</geometry>
 				<material name="yellow">
@@ -37,5 +37,5 @@
 				<origin xyz="0.050 -.028 0" rpy="0 0 -0.52"/>
 				<geometry>
-                    <mesh filename="package://hera_description/meshes/gripper_meshes/visual/link_1.dae" scale= "0.6 0.6 0.6" />
+                    <mesh filename="package://hera_description/meshes/gripper_meshes/visual/link_1.dae" scale= "0.7 0.7 0.7" />
 				</geometry>
 				<material name="light grey"/>
@@ -44,5 +44,5 @@
 				<origin xyz="0.050 -.028 0" rpy="0 0 -0.52"/>
 				<geometry>
-                    <mesh filename="package://hera_description/meshes/gripper_meshes/collision/link_1.STL" scale= "0.6 0.6 0.6" />
+                    <mesh filename="package://hera_description/meshes/gripper_meshes/collision/link_1.STL" scale= "0.7 0.7 0.7" />
 				</geometry>
 				<material name="yellow"/>
@@ -63,5 +63,5 @@
 				<origin xyz="0.039 0 0.0075" rpy="0 0 0"/>
 				<geometry>
-                    <mesh filename="package://hera_description/meshes/gripper_meshes/visual/link_2.dae" scale= "0.6 0.6 0.6" />
+                    <mesh filename="package://hera_description/meshes/gripper_meshes/visual/link_2.dae" scale= "0.7 0.7 0.7" />
 				</geometry>
 				<material name="light grey"/>
@@ -70,5 +70,5 @@
 				<origin xyz="0.039 0 0.0075" rpy="0 0 0"/>
 				<geometry>
-                    <mesh filename="package://hera_description/meshes/gripper_meshes/collision/link_2.STL" scale= "0.6 0.6 0.6" />
+                    <mesh filename="package://hera_description/meshes/gripper_meshes/collision/link_2.STL" scale= "0.7 0.7 0.7" />
 				</geometry>
 				<material name="yellow"/>
@@ -84,5 +84,5 @@
 				<origin xyz="0 0 0" rpy="0 0 0.52"/>
 				<geometry>
-                    <mesh filename="package://hera_description/meshes/gripper_meshes/visual/link_3.dae" scale= "0.6 0.6 0.6" />
+                    <mesh filename="package://hera_description/meshes/gripper_meshes/visual/link_3.dae" scale= "0.7 0.7 0.7" />
 				</geometry>
 				<material name="light grey"/>
@@ -91,5 +91,5 @@
 				<origin xyz="0 0 0" rpy="0 0 0.52"/>
 				<geometry>
-                    <mesh filename="package://hera_description/meshes/gripper_meshes/collision/link_3.STL" scale= "0.6 0.6 0.6" />
+                    <mesh filename="package://hera_description/meshes/gripper_meshes/collision/link_3.STL" scale= "0.7 0.7 0.7" />
 				</geometry>
 				<material name="yellow"/>
@@ -107,6 +107,6 @@
 			<child link="${prefix}link_1"/>
 			<axis xyz="0 0 1"/>
-			<origin xyz="0.0005 0.01 0" rpy="0 0 0"/>
-			<limit lower="-0.6503" upper="0.3159" effort="100" velocity="100"/>
+			<origin xyz="0.01 0.0 0" rpy="0 0 0"/>
+			<limit lower="-0.6503" upper="1.0" effort="100" velocity="100"/>
 		</joint>
 		<joint name="${prefix}joint_2" type="revolute">
@@ -114,6 +114,6 @@
 			<child link="${prefix}link_2"/>
 			<axis xyz="0 0 1"/>
-			<origin xyz="0.035 -0.025 0" rpy="0 0 -0.52"/>
-			<limit lower="-0.2787" upper="0.5960" effort="100" velocity="100"/>
+			<origin xyz="0.04 -0.025 0" rpy="0 0 -0.52"/>
+			<limit lower="-0.2787" upper="1.0" effort="100" velocity="100"/>
 		</joint>
 		<joint name="${prefix}joint_3" type="fixed">

File: hera_description/urdf/actuators/torso.urdf.xacro (robot description, xacro)
@@ -13,6 +13,6 @@
   <xacro:property name="small_box_size_z"  value="0.30"/>
   <xacro:property name="head_plat_mass"    value="0.10"/>
-  <xacro:property name="head_plat_size_x"  value="0.25"/>
-  <xacro:property name="head_plat_size_y"  value="0.30"/>
+  <xacro:property name="head_plat_size_x"  value="0.35"/>
+  <xacro:property name="head_plat_size_y"  value="${base_size_y}"/>
   <xacro:property name="head_plat_size_z"  value="0.05"/>
   <xacro:property name="pole_mass"         value="0.20"/>
@@ -20,5 +20,5 @@
   <xacro:property name="pole_size_y"       value="0.06"/>
   <xacro:property name="pole_size_z"       value="1.00"/>
-  <xacro:property name="sensor_plat_mass"             value="0.00001"/>
+  <xacro:property name="sensor_plat_mass"             value="0.01"/>
   <xacro:property name="sensor_plat_size_x"           value="0.10"/>
   <xacro:property name="sensor_plat_size_y"           value="0.12"/>
@@ -43,11 +43,11 @@
         <origin xyz="0.15 0 -0.35" rpy="0 0 0"/>
       </xacro:create_box>
-      <!-- <xacro:create_box
+      <xacro:create_box
         m="${head_plat_mass}"
         x="${head_plat_size_x}"
         y="${head_plat_size_y}"
         z="${head_plat_size_z}">
-        <origin xyz="-0.08 0 0.475" rpy="0 0 0"/>
-      </xacro:create_box> -->
+        <origin xyz="-0.06 0 0.475" rpy="0 0 0"/>
+      </xacro:create_box>
       <xacro:create_box
         m="${pole_mass}"
@@ -106,5 +106,5 @@
       <parent link="${name}"/>
       <child link="${name}_sensor_plat"/>
-      <axis xyz="0 1 0"/>
+      <axis xyz="0 1 0"/> -->
       <limit effort="${torso_sensor_plat_effort}" velocity="${torso_sensor_plat_velocity}"
         lower="0.0" upper="1.57"/>

File: hera_description/urdf/simulation/control.gazebo.xacro (robot description, xacro)
@@ -3,5 +3,4 @@
   <gazebo>
     <plugin name="gazebo_ros_control" filename="libgazebo_ros_control.so"/>
-    <rosparam file="$(find hera_description)/config/yaml/gazebo_ros_control_params.yaml" command="load"/>
   </gazebo>
 </robot>

Commit message: Increased base mass

File: hera_description/urdf/actuators/base.urdf.xacro (robot description, xacro)
@@ -4,5 +4,5 @@
        xmlns:interface="http://playerstage.sourceforge.net/gazebo/xmlschema/#interface"
        xmlns:xacro="http://ros.org/wiki/xacro">
-  <xacro:property name="base_mass"      value="20.0"/>
+  <xacro:property name="base_mass"      value="100.0"/>
   <xacro:property name="base_size_x"    value="0.50"/>
   <xacro:property name="base_size_y"    value="0.30"/>
