Commit message: Added manipulator

File: hera_description/robots/hera_full.urdf.xacro (robot description, xacro)
@@ -13,6 +13,7 @@
   <!-- actuators -->
   <xacro:include filename="$(find hera_description)/urdf/actuators/base.urdf.xacro" />
-  <xacro:include filename="$(find hera_description)/urdf/actuators/torso.urdf.xacro" />
+  <xacro:include filename="/home/guilherme/ws_moveit/src/hera_description/urdf/actuators/torso.urdf.xacro" />
   <xacro:include filename="$(find hera_description)/urdf/actuators/head.urdf.xacro" />
+  <xacro:include filename="/home/guilherme/ws_moveit/src/hera_description/urdf/actuators/manip.urdf.xacro" />
   <!-- sensors -->
   <xacro:include filename="$(find hera_description)/urdf/sensors/hokuyo_utm.urdf.xacro"/>
@@ -66,4 +67,12 @@
     <origin xyz="0.05 0 0.1" rpy="0 0 0" />
   </xacro:kinect_one>
+  <!--torso suporte-->
+  <xacro:create_suporte_link
+    parent="torso"/>
+  <!--torso encosto-->
+  <xacro:create_encosto_link
+    parent="torso"/>
+  <!-- manip -->
+  <xacro:manip/>
 <!-- ####################################################################### -->
 <!-- ####################### gazebo extensions ##############################-->

File: hera_description/urdf/actuators/torso.urdf.xacro (robot description, xacro)
@@ -71,4 +71,11 @@
         </geometry>
       </visual>
+      <collision>
+        <origin xyz="0 0 -0.5" rpy="0 0 0"/>
+        <material name="dark_grey"/>
+        <geometry>
+          <mesh filename="package://hera_description/meshes/torso.stl"/>
+        </geometry>
+      </collision>
     </link>
     <!-- sensor plat -->
@@ -95,11 +102,11 @@
     </joint>
     <!-- should be revolute -->
-    <joint name="joint_${name}to${name}_sensor_plat" type="revolute">
+    <joint name="joint_${name}_to_${name}_sensor_plat" type="revolute">
       <origin xyz="0.09 0 0.46" rpy="0 0 0"/> <!-- rpy="0 0 0" -->
       <parent link="${name}"/>
       <child link="${name}_sensor_plat"/>
-      <axis xyz="0 1 0"/>
+      <axis xyz="0 1 0"/> -->
       <limit effort="${torso_sensor_plat_effort}" velocity="${torso_sensor_plat_velocity}"
-        lower="-1.0216" upper="-0.6592" />
+        lower="0.0" upper="1.57"/>
     </joint>
     <!-- <transmission name="tran_${name}_sensor_plat">
@@ -114,3 +121,61 @@
     </transmission> -->
   </xacro:macro>
+  <!--suporte_link-->
+  <xacro:macro name="create_suporte_link" params="parent">
+    <link name="suporte_link">
+      <visual>
+        <origin xyz="0 0 0" rpy="0 0 0" />
+        <geometry>
+          <mesh filename="package://hera_description/meshes/manip_meshes/suporte_link.STL"/>
+        </geometry>
+        <material name="grey">
+          <color rgba="0.792156862745098 0.819607843137255 0.933333333333333 1" />
+        </material>
+      </visual>
+      <collision>
+        <origin xyz="0 0 0" rpy="0 0 0" />
+        <geometry>
+          <mesh filename="package://hera_description/meshes/manip_meshes/suporte_link.STL"/>
+        </geometry>
+      </collision>
+      <xacro:inertial_suporte_link mass="0.659217140679788"/>
+    </link>
+    <!--suporte_joint-->
+    <joint name="suporte_joint" type="fixed">
+      <origin xyz="0.04525 0 0.0285" rpy="0 0 0" />
+      <parent link="${parent}" />
+      <child link="suporte_link" />
+      <axis xyz="0 0 0" />
+      <limit lower="0" upper="0" effort="0" velocity="0" />
+    </joint>
+  </xacro:macro>
+  <!--encosto_link-->
+  <xacro:macro name="create_encosto_link" params="parent">
+    <link name="encosto_link">
+      <visual>
+        <origin xyz="0 0 0" rpy="0 0 0" />
+        <geometry>
+          <mesh filename="package://hera_description/meshes/manip_meshes/encosto_link.STL"/>
+        </geometry>
+        <material name="grey">
+          <color rgba="0.898039215686275 0.917647058823529 0.929411764705882 1" />
+        </material>
+      </visual>
+      <collision>
+        <origin xyz="0 0 0" rpy="0 0 0" />
+        <geometry>
+          <mesh filename="package://hera_description/meshes/manip_meshes/encosto_link.STL"/>
+        </geometry>
+      </collision>
+      <xacro:inertial_base_link mass="0.0709912944888601"/>
+    </link>
+    <!--encosto_joint-->
+    <joint name="encosto_joint" type="fixed">
+      <origin xyz="0.028 0.0066709 0.053" rpy="0 0 0" />
+      <parent link="${parent}" />
+      <child link="encosto_link" />
+      <axis xyz="0 0 0" />
+      <limit effort="0" velocity="0" />
+    </joint>
+  </xacro:macro>
 </robot>

File: hera_description/urdf/simulation/asus_xtion.gazebo.xacro (robot description, xacro)
@@ -11,6 +11,6 @@
             <image>
               <format>R8G8B8</format>
-              <width>${640}</width>
-              <height>${480}</height>
+              <width>${640/20}</width>
+              <height>${480/20}</height>
             </image>
             <clip>

File: hera_description/urdf/simulation/kinect_one.gazebo.xacro (robot description, xacro)
@@ -10,6 +10,6 @@
                 <image>
                   <format>R8G8B8</format>
-                  <width>${640}</width>
-                  <height>${480}</height>
+                  <width>${640/20}</width>
+                  <height>${480/20}</height>
                 </image>
                 <clip>

Commit message: Added meshes and changed xacro to change Hera's gripper

File: hera_description/robots/hera_full.urdf.xacro (robot description, xacro)
@@ -29,4 +29,5 @@
   <xacro:include filename="$(find hera_description)/urdf/simulation/asus_xtion.gazebo.xacro" />
   <xacro:include filename="$(find hera_description)/urdf/simulation/kinect_one.gazebo.xacro" />
+  <xacro:include filename="$(find hera_description)/urdf/simulation/manip.gazebo.xacro" />
 <!-- ####################################################################### -->
 <!-- ######################## robot parts ################################## -->
@@ -101,3 +102,5 @@
     reference="kinect_one"
     update_rate="30"/>
+  <!-- manip_plugin -->
+  <xacro:gazebo_manip/>
 </robot>

File: hera_description/urdf/actuators/base.urdf.xacro (robot description, xacro)
@@ -4,5 +4,5 @@
        xmlns:interface="http://playerstage.sourceforge.net/gazebo/xmlschema/#interface"
        xmlns:xacro="http://ros.org/wiki/xacro">
-  <xacro:property name="base_mass"      value="99.9"/>
+  <xacro:property name="base_mass"      value="20.0"/>
   <xacro:property name="base_size_x"    value="0.50"/>
   <xacro:property name="base_size_y"    value="0.30"/>

File: hera_description/urdf/actuators/manip.urdf.xacro (robot description, xacro)
@@ -2,4 +2,6 @@
 <robot xmlns:xacro="http://www.ros.org/wiki/xacro" name="hera_description">
 <xacro:include filename="$(find hera_description)/urdf/manip_prop.urdf.xacro"/>
+<xacro:include filename="$(find hera_description)/urdf/simulation/manip_transmission.xacro"/>
+<xacro:include filename="$(find hera_description)/urdf/actuators/gripper/robotiq-3f-gripper_articulated_macro.xacro"/>
 <!--base_link-->
   <xacro:macro name="create_base_link">
@@ -81,9 +83,9 @@
     <!--joint_2-->
     <joint name="joint_2" type="revolute">
-      <origin xyz="0.048 0 0.02285" rpy="3.1416 -1.1781 -3.1416" />
+      <origin xyz="0.048 0 0.02285" rpy="3.1416 -2 -3.1416" />
       <parent link="link_1" />
       <child link="link_2" />
       <axis xyz="0 1 0" />
-      <limit lower="-1.0847" upper="3.14" effort="8" velocity="5" />
+      <limit lower="-2.355" upper="3.14" effort="8" velocity="5" />
     </joint>
   </xacro:macro>
@@ -181,5 +183,5 @@
         <origin xyz="0 0 0" rpy="0 0 0"/>
         <geometry>
-          <mesh  filename="package://hera_description/meshes/manip_meshes/link_6.STL" />
+          <mesh  filename="package://hera_description/meshes/manip_meshes/link_6.STL" scale="0.1 0.1 0.1" />
         </geometry>
         <material name="dark_grey">
@@ -190,5 +192,5 @@
         <origin xyz="0 0 0" rpy="0 0 0"/>
         <geometry>
-          <mesh filename="package://hera_description/meshes/manip_meshes/link_6_col.STL" />
+          <mesh filename="package://hera_description/meshes/manip_meshes/link_6_col.STL" scale="0.1 0.1 0.1" />
         </geometry>
         </collision>
@@ -202,118 +204,4 @@
       <axis xyz="0 -1 0" />
       <limit lower="-2.6232" upper="1.8262" effort="8" velocity="5" />
-    </joint>
-  </xacro:macro>
-<!--link_7-->
-  <xacro:macro name="create_link_7">
-    <link name="link_7">
-      <visual>
-        <origin xyz="0 0 0" rpy="0 0 0" />
-        <geometry>
-          <mesh filename="package://hera_description/meshes/manip_meshes/link_7.STL"/>
-        </geometry>
-        <material name="dark_grey">
-          <color rgba="0.898039215686275 0.917647058823529 0.929411764705882 1" />
-        </material>
-      </visual>
-      <collision>
-        <origin xyz="0 0 0" rpy="0 0 0" />
-        <geometry>
-          <mesh filename="package://hera_description/meshes/manip_meshes/link_7_col.STL"/>
-        </geometry>
-      </collision>
-      <xacro:inertial_link_7 mass="0.0392347304267543"/>
-    </link>
-    <!-- joint 7 -->
-    <joint name="joint_7" type="revolute">
-      <origin xyz="0.061 0.02125 0" rpy="0 0 0" />
-      <parent link="link_6" />
-      <child  link="link_7" />
-      <axis xyz="0 0 1" />
-      <limit lower="-0.6454" upper="1.5600" effort="8" velocity="5" />
-    </joint>
-  </xacro:macro>
-<!--link_end7-->
-  <xacro:macro name="create_link_end7">
-    <link name="link_end7">
-      <visual>
-        <origin xyz="0 0 0" rpy="0 0 0" />
-        <geometry>
-          <mesh filename="package://hera_description/meshes/manip_meshes/link_end7.STL"/>
-        </geometry>
-        <material name="white">
-          <color rgba="0.898039215686275 0.917647058823529 0.929411764705882 1" />
-        </material>
-      </visual>
-      <collision>
-        <origin xyz="0 0 0" rpy="0 0 0" />
-        <geometry>
-          <mesh filename="package://hera_description/meshes/manip_meshes/link_end7.STL"/>
-        </geometry>
-      </collision>
-      <xacro:inertial_link_end7 mass="0.0535201883186937"/>
-    </link>
-    <!--joint_end7-->
-    <joint name="joint_end7" type="fixed">
-      <origin xyz="0.066179 -0.02125 0" rpy="0 0 0" />
-      <parent link="link_7" />
-      <child link="link_end7" />
-      <axis xyz="0 0 0" />
-    </joint>
-  </xacro:macro>
-<!--link_8-->
-  <xacro:macro name="create_link_8">
-    <link name="link_8">
-      <visual>
-        <origin xyz="0 0 0" rpy="0 0 0" />
-        <geometry>
-          <mesh filename="package://hera_description/meshes/manip_meshes/link_8.STL" />
-        </geometry>
-        <material name="dark_grey">
-          <color rgba="0.898039215686275 0.917647058823529 0.929411764705882 1" />
-        </material>
-      </visual>
-      <collision>
-        <origin xyz="0 0 0" rpy="0 0 0" />
-        <geometry>
-          <mesh filename="package://hera_description/meshes/manip_meshes/link_8_col.STL" />
-        </geometry>
-      </collision>
-      <xacro:inertial_link_8 mass="0.0392347308783591"/>
-    </link>
-    <!--joint_8-->
-    <joint name="joint_8" type="revolute">
-      <origin xyz="0.061 -0.02125 0" rpy="0 0 0" />
-      <parent link="link_6" />
-      <child link="link_8" />
-      <axis xyz="0 0 1" />
-      <limit lower="-1.5600" upper="0.6454" effort="8" velocity="5" />
-    </joint>
-  </xacro:macro>
-<!--link_end8-->
-  <xacro:macro name="create_link_end8">
-    <link name="link_end8">
-      <visual>
-        <origin xyz="0 0 0" rpy="0 0 0" />
-        <geometry>
-          <mesh filename="package://hera_description/meshes/manip_meshes/link_end8.STL" />
-        </geometry>
-        <material name="white">
-          <color rgba="0.898039215686275 0.917647058823529 0.929411764705882 1" />
-        </material>
-      </visual>
-      <collision>
-        <origin xyz="0 0 0" rpy="0 0 0" />
-        <geometry>
-          <mesh filename="package://hera_description/meshes/manip_meshes/link_end8.STL" />
-        </geometry>
-      </collision>
-      <xacro:inertial_link_end8 mass="0.0535202013033793"/>
-    </link>
-    <!--joint_end8-->
-    <joint name="joint_end8" type="fixed">
-      <origin xyz="0.0661786041848968 0.0212499999999973 0" rpy="0 0 0" />
-      <parent link="link_8" />
-      <child link="link_end8" />
-      <axis xyz="0 0 0" />
     </joint>
   </xacro:macro>
@@ -333,12 +221,8 @@
     <!--link_6-->
     <xacro:create_link_6/>
-    <!--link_7-->
-    <xacro:create_link_7/>
-    <!--link_end7-->
-    <xacro:create_link_end7/>
-    <!--link_8-->
-    <xacro:create_link_8/>
-    <!--link_end8-->
-    <xacro:create_link_end8/>
+    <!-- Gripper -->
+    <xacro:robotiq-3f-gripper_articulated prefix=""/>
+    <!--Transmission-->
+    <xacro:manip_transmission/>
   </xacro:macro>
 </robot>

File: hera_description/urdf/actuators/torso.urdf.xacro (robot description, xacro)
@@ -102,23 +102,23 @@
     </joint>
     <!-- should be revolute -->
-    <!-- should be revolute -->
-    <joint name="joint_${name}_to_${name}_sensor_plat" type="fixed">
+    <joint name="joint_${name}_to_${name}_sensor_plat" type="revolute">
       <origin xyz="0.09 0 0.46" rpy="0 0 0"/> <!-- rpy="0 0 0" -->
       <parent link="${name}"/>
       <child link="${name}_sensor_plat"/>
-      <!-- <axis xyz="0 1 0"/> -->
-      <!-- <limit effort="${torso_sensor_plat_effort}" velocity="${torso_sensor_plat_velocity}"
-        lower="0.0" upper="${M_PI/2}"/> -->
+      <axis xyz="0 1 0"/> -->
+      <limit effort="${torso_sensor_plat_effort}" velocity="${torso_sensor_plat_velocity}"
+        lower="0.0" upper="1.57"/>
     </joint>
-    <!-- <transmission name="tran_${name}_sensor_plat">
+    <!-- Transmission to Gazebo Plugin -->
+    <transmission name="trans_kinect">
       <type>transmission_interface/SimpleTransmission</type>
-      <joint name="joint_${name}_to_${name}_sensor_plat">
+      <joint name="joint_torso_to_torso_sensor_plat">
         <hardwareInterface>hardware_interface/EffortJointInterface</hardwareInterface>
       </joint>
-      <actuator name="motor_${name}_sensor_plat">
+      <actuator name="kinect_motor">
         <hardwareInterface>hardware_interface/EffortJointInterface</hardwareInterface>
         <mechanicalReduction>1</mechanicalReduction>
       </actuator>
-    </transmission> -->
+    </transmission>
   </xacro:macro>
   <!--suporte_link-->

File: hera_description/urdf/simulation/colors.gazebo.xacro (robot description, xacro)
@@ -1,4 +1,5 @@
 <?xml version="1.0"?>
 <robot xmlns:xacro="http://ros.org/wiki/xacro">
+  <!-- manip colors -->
   <gazebo reference="base"><material>Gazebo/Black</material></gazebo>
   <gazebo reference="base_wheelFR"><material>Gazebo/White</material></gazebo>
@@ -9,3 +10,25 @@
   <gazebo reference="torso_sensor_plat"><material>Gazebo/DarkGray</material></gazebo>
   <gazebo reference="head"><material>Gazebo/Gray</material></gazebo>
+  <!-- manip colors -->
+  <gazebo reference="base_link"><material>Gazebo/Gray</material></gazebo>
+  <gazebo reference="link_1"><material>Gazebo/Gray</material></gazebo>
+  <gazebo reference="link_2"><material>Gazebo/Gray</material></gazebo>
+  <gazebo reference="link_3"><material>Gazebo/Gray</material></gazebo>
+  <gazebo reference="link_4"><material>Gazebo/Gray</material></gazebo>
+  <gazebo reference="link_5"><material>Gazebo/Gray</material></gazebo>
+  <gazebo reference="link_6"><material>Gazebo/Gray</material></gazebo>
+  <gazebo reference="palm"><material>Gazebo/White</material></gazebo>
+  <gazebo reference="tool0"><material>Gazebo/White</material></gazebo>
+  <gazebo reference="finger_1_link_0"><material>Gazebo/White</material></gazebo>
+  <gazebo reference="finger_1_link_1"><material>Gazebo/White</material></gazebo>
+  <gazebo reference="finger_1_link_2"><material>Gazebo/White</material></gazebo>
+  <gazebo reference="finger_1_link_3"><material>Gazebo/White</material></gazebo>
+  <gazebo reference="finger_2_link_0"><material>Gazebo/White</material></gazebo>
+  <gazebo reference="finger_2_link_1"><material>Gazebo/White</material></gazebo>
+  <gazebo reference="finger_2_link_2"><material>Gazebo/White</material></gazebo>
+  <gazebo reference="finger_2_link_3"><material>Gazebo/White</material></gazebo>
+  <gazebo reference="finger_middle_link_0"><material>Gazebo/White</material></gazebo>
+  <gazebo reference="finger_middle_link_1"><material>Gazebo/White</material></gazebo>
+  <gazebo reference="finger_middle_link_2"><material>Gazebo/White</material></gazebo>
+  <gazebo reference="finger_middle_link_3"><material>Gazebo/White</material></gazebo>
 </robot>

File: hera_description/urdf/simulation/kinect_one.gazebo.xacro (robot description, xacro)
@@ -10,6 +10,6 @@
                 <image>
                   <format>R8G8B8</format>
-                  <width>${640}</width>
-                  <height>${480}</height>
+                  <width>${640/20}</width>
+                  <height>${480/20}</height>
                 </image>
                 <clip>
@@ -42,4 +42,10 @@
           </sensor>
         </gazebo>
+        <gazebo>
+            <plugin name="gazebo_ros_control" filename="libgazebo_ros_control.so">
+            <robotNamespace>/kinect</robotNamespace>
+            <robotSimType>gazebo_ros_control/DefaultRobotHWSim</robotSimType>
+            </plugin>
+        </gazebo>
     </xacro:macro>
   </robot>

Commit message: Added pid gains to kinect and manip controllers

File: hera_description/robots/hera_full.urdf.xacro (robot description, xacro)
@@ -63,9 +63,9 @@
   </xacro:xtion>
   <!-- torso pointcloud front: kinect_one -->
-  <xacro:kinect_one
+  <!-- <xacro:kinect_one
     name="kinect_one"
     parent="torso_sensor_plat">
     <origin xyz="0.05 0 0.1" rpy="0 0 0" />
-  </xacro:kinect_one>
+  </xacro:kinect_one> -->
   <!--torso suporte-->
   <xacro:create_suporte_link

File: hera_description/urdf/actuators/base.urdf.xacro (robot description, xacro)
@@ -4,5 +4,5 @@
        xmlns:interface="http://playerstage.sourceforge.net/gazebo/xmlschema/#interface"
        xmlns:xacro="http://ros.org/wiki/xacro">
-  <xacro:property name="base_mass"      value="20.0"/>
+  <xacro:property name="base_mass"      value="50.0"/>
   <xacro:property name="base_size_x"    value="0.50"/>
   <xacro:property name="base_size_y"    value="0.30"/>

File: hera_description/urdf/actuators/torso.urdf.xacro (robot description, xacro)
@@ -13,6 +13,6 @@
   <xacro:property name="small_box_size_z"  value="0.30"/>
   <xacro:property name="head_plat_mass"    value="0.10"/>
-  <xacro:property name="head_plat_size_x"  value="0.35"/>
-  <xacro:property name="head_plat_size_y"  value="${base_size_y}"/>
+  <xacro:property name="head_plat_size_x"  value="0.25"/>
+  <xacro:property name="head_plat_size_y"  value="0.30"/>
   <xacro:property name="head_plat_size_z"  value="0.05"/>
   <xacro:property name="pole_mass"         value="0.20"/>
@@ -20,5 +20,5 @@
   <xacro:property name="pole_size_y"       value="0.06"/>
   <xacro:property name="pole_size_z"       value="1.00"/>
-  <xacro:property name="sensor_plat_mass"             value="0.01"/>
+  <xacro:property name="sensor_plat_mass"             value="0.0001"/>
   <xacro:property name="sensor_plat_size_x"           value="0.10"/>
   <xacro:property name="sensor_plat_size_y"           value="0.12"/>
@@ -43,11 +43,11 @@
         <origin xyz="0.15 0 -0.35" rpy="0 0 0"/>
       </xacro:create_box>
-      <xacro:create_box
+      <!-- <xacro:create_box
         m="${head_plat_mass}"
         x="${head_plat_size_x}"
         y="${head_plat_size_y}"
         z="${head_plat_size_z}">
-        <origin xyz="-0.06 0 0.475" rpy="0 0 0"/>
-      </xacro:create_box>
+        <origin xyz="-0.08 0 0.475" rpy="0 0 0"/>
+      </xacro:create_box> -->
       <xacro:create_box
         m="${pole_mass}"
@@ -106,5 +106,5 @@
       <parent link="${name}"/>
       <child link="${name}_sensor_plat"/>
-      <axis xyz="0 1 0"/> -->
+      <axis xyz="0 1 0"/>
       <limit effort="${torso_sensor_plat_effort}" velocity="${torso_sensor_plat_velocity}"
         lower="0.0" upper="1.57"/>

File: hera_description/urdf/simulation/control.gazebo.xacro (robot description, xacro)
@@ -3,4 +3,5 @@
   <gazebo>
     <plugin name="gazebo_ros_control" filename="libgazebo_ros_control.so"/>
+    <rosparam file="$(find hera_description)/config/yaml/gazebo_ros_control_params.yaml" command="load"/>
   </gazebo>
 </robot>

Commit message: Kinect controller glitch fixed

File: hera_description/robots/hera_full.urdf.xacro (robot description, xacro)
@@ -63,9 +63,9 @@
   </xacro:xtion>
   <!-- torso pointcloud front: kinect_one -->
-  <!-- <xacro:kinect_one
+  <xacro:kinect_one
     name="kinect_one"
     parent="torso_sensor_plat">
     <origin xyz="0.05 0 0.1" rpy="0 0 0" />
-  </xacro:kinect_one> -->
+  </xacro:kinect_one>
   <!--torso suporte-->
   <xacro:create_suporte_link

File: hera_description/urdf/actuators/torso.urdf.xacro (robot description, xacro)
@@ -20,5 +20,5 @@
   <xacro:property name="pole_size_y"       value="0.06"/>
   <xacro:property name="pole_size_z"       value="1.00"/>
-  <xacro:property name="sensor_plat_mass"             value="0.0001"/>
+  <xacro:property name="sensor_plat_mass"             value="0.00001"/>
   <xacro:property name="sensor_plat_size_x"           value="0.10"/>
   <xacro:property name="sensor_plat_size_y"           value="0.12"/>
