Commit message: Added plugin to contact sensor

File: hera_description/robots/hera_full.urdf.xacro (robot description, xacro)
@@ -104,3 +104,92 @@
   <!-- manip_plugin -->
   <xacro:gazebo_manip/>
+<!-- ####################################################################### -->
+<!-- ####################### gazebo sensors #################################-->
+<!-- ####################################################################### -->
+  <gazebo reference="link_6">
+    <turnGravityOff>true</turnGravityOff>
+    <selfCollide>false</selfCollide>
+    <sensor type="contact" name="palm_contactsensor_sensor">
+      <update_rate>100.0</update_rate>
+      <contact>
+        <collision>link_6_fixed_joint_lump__palm_collision_1</collision>
+      </contact>
+      <plugin name="palm_plugin" filename="libgazebo_ros_bumper.so">
+        <alwaysOn>true</alwaysOn>
+        <frameName>link_6</frameName>
+        <updateRate>100.0</updateRate>
+        <bumperTopicName>link_6_bumper</bumperTopicName>
+      </plugin>
+    </sensor>
+    <mu1 value="500.0" />
+    <mu2 value="500.0" />
+    <kp  value="10000000.0" />
+    <kd  value="1.0" />
+  </gazebo>
+<!--FINGER MIDDLE LINK 3 SENSOR-->
+  <gazebo reference="finger_middle_link_3">
+    <turnGravityOff>true</turnGravityOff>
+    <selfCollide>false</selfCollide>
+    <sensor type="contact" name="finger_middle_link_3_contactsensor_sensor">
+      <update_rate>100.0</update_rate>
+      <contact>
+        <collision>finger_middle_link_3_collision</collision>
+      </contact>
+      <plugin name="finger_middle_link_3_plugin" filename="libgazebo_ros_bumper.so">
+        <alwaysOn>true</alwaysOn>
+        <frameName>finger_middle_link_3</frameName>
+        <updateRate>100.0</updateRate>
+        <bumperTopicName>finger_middle_link_3_bumper</bumperTopicName>
+      </plugin>
+    </sensor>
+    <mu1 value="500.0" />
+    <mu2 value="500.0" />
+    <kp  value="10000000.0" />
+    <kd  value="1.0" />
+    <provideFeedback value="true"/>
+  </gazebo>
+<!--FINGER 2 LINK 3 SENSOR-->
+  <gazebo reference="base_wheelFL">
+    <turnGravityOff>true</turnGravityOff>
+    <selfCollide>false</selfCollide>
+    <sensor type="contact" name="base_wheelFL_contactsensor_sensor">
+      <update_rate>100.0</update_rate>
+      <contact>
+        <collision>base_wheelFL_collision</collision>
+      </contact>
+      <plugin name="base_wheelFL_plugin" filename="libgazebo_ros_bumper.so">
+        <alwaysOn>true</alwaysOn>
+        <frameName>base_wheelFL</frameName>
+        <updateRate>100.0</updateRate>
+        <bumperTopicName>base_wheelFL_bumper</bumperTopicName>
+      </plugin>
+    </sensor>
+    <mu1 value="500.0" />
+    <mu2 value="500.0" />
+    <kp  value="10000000.0" />
+    <kd  value="1.0" />
+    <provideFeedback value="true"/>
+  </gazebo>
+  <!--FINGER 1 LINK 3 SENSOR-->
+  <gazebo reference="finger_1_link_3">
+    <turnGravityOff>true</turnGravityOff>
+    <selfCollide>false</selfCollide>
+    <sensor type="contact" name="finger_1_link_3_contactsensor_sensor">
+      <update_rate>100.0</update_rate>
+      <contact>
+        <collision>finger_1_link_2_fixed_joint_lump__finger_1_link_3_collision_1</collision>
+      </contact>
+      <plugin name="finger_1_link_3_plugin" filename="libgazebo_ros_bumper.so">
+        <alwaysOn>true</alwaysOn>
+        <frameName>finger_1_link_3</frameName>
+        <updateRate>100.0</updateRate>
+        <bumperTopicName>finger_1_link_3_bumper</bumperTopicName>
+      </plugin>
+    </sensor>
+    <mu1 value="500.0" />
+    <mu2 value="500.0" />
+    <kp  value="10000000.0" />
+    <kd  value="1.0" />
+    <provideFeedback value="true"/>
+  </gazebo>
 </robot>

Commit message: Added gripper contact sensors

File: hera_description/robots/hera_full.urdf.xacro (robot description, xacro)
@@ -21,4 +21,5 @@
   <xacro:include filename="$(find hera_description)/urdf/sensors/asus_xtion.urdf.xacro"/>
   <xacro:include filename="$(find hera_description)/urdf/sensors/kinect_one.urdf.xacro"/>
+  <xacro:include filename="$(find hera_description)/urdf/sensors/gripper_contact_sensors.urdf.xacro"/>
   <!-- simulation -->
   <xacro:include filename="$(find hera_description)/urdf/simulation/colors.gazebo.xacro" />
@@ -104,3 +105,49 @@
   <!-- manip_plugin -->
   <xacro:gazebo_manip/>
+  <!-- gripper_contact_sensors -->
+  <xacro:gripper_contact_sensors/>
+<!-- ####################################################################### -->
+<!-- ####################### gazebo sensors #################################-->
+<!-- ####################################################################### -->
+  <!-- <gazebo reference="link_6">
+    <turnGravityOff>true</turnGravityOff>
+    <selfCollide>false</selfCollide>
+    <sensor type="contact" name="palm_contactsensor_sensor">
+      <update_rate>100.0</update_rate>
+      <contact>
+        <collision>link_6_fixed_joint_lump__palm_collision_1</collision>
+      </contact>
+      <plugin name="palm_plugin" filename="libgazebo_ros_bumper.so">
+        <alwaysOn>true</alwaysOn>
+        <frameName>link_6</frameName>
+        <updateRate>100.0</updateRate>
+        <bumperTopicName>link_6_bumper</bumperTopicName>
+      </plugin>
+    </sensor>
+    <mu1 value="500.0" />
+    <mu2 value="500.0" />
+    <kp  value="10000000.0" />
+    <kd  value="1.0" />
+  </gazebo> -->
+  <!-- FINGER 1 LINK 3 SENSOR
+  <gazebo reference="finger_1_link_3">
+    <turnGravityOff>true</turnGravityOff>
+    <selfCollide>false</selfCollide>
+    <sensor type="contact" name="finger_1_link_3_contactsensor_sensor">
+      <alwaysOn>true</alwaysOn>
+      <update_rate>100.0</update_rate>
+      <contact>
+        <collision>finger_1_link_2_fixed_joint_lump__finger_1_link_3_collision_1</collision>
+      </contact>
+      <plugin name="finger_1_link_3_plugin" filename="libgazebo_ros_bumper.so">
+        <bumperTopicName>finger_1_link_3_bumper</bumperTopicName>
+        <frameName>finger_1_link_3</frameName>
+      </plugin>
+    </sensor>
+    <mu1 value="500.0" />
+    <mu2 value="500.0" />
+    <kp  value="10000000.0" />
+    <kd  value="1.0" />
+    <provideFeedback value="true"/>
+  </gazebo> -->
 </robot>

File: hera_description/urdf/actuators/head.urdf.xacro (robot description, xacro)
@@ -53,5 +53,5 @@
       </visual>
     </link>
-    <joint name="joint_${parent}_to_${name}" type="revolute">
+    <joint name="joint_${parent}_to_${name}" type="fixed">
       <origin xyz="-0.06 0 ${(pole_size_z/2)+(head_base_length)+(head_box_size_z/2)}" rpy="0 0 0"/>
       <child link="${name}"/>
@@ -60,5 +60,5 @@
       <limit effort="${head_effort}" velocity="${head_velocity}" lower="-${M_PI/2}" upper="${M_PI/2}"/>
     </joint>
-    <transmission name="tran_${name}">
+    <!-- <transmission name="tran_${name}">
       <type>transmission_interface/SimpleTransmission</type>
       <joint name="joint_${parent}_to_${name}">
@@ -69,5 +69,5 @@
         <mechanicalReduction>1</mechanicalReduction>
       </actuator>
-    </transmission>
+    </transmission> -->
   </xacro:macro>
 </robot>
